Commit message: gnss location

File: src/mapping/lio-sam/launch/include/config/cicv_robot.urdf.xacro (robot description, xacro)
@@ -25,10 +25,3 @@
     <origin xyz="0.0 0.0 0.0" rpy="0.0 0.0 0.0" />
   </joint>
-  <!-- Sensor: odometry -->
-  <link name="ego_vehicle/odometry"></link>
-  <joint name="odometry_joint" type="fixed">
-    <parent link="ego_vehicle" />
-    <child link="ego_vehicle/odometry" />
-    <origin xyz="0.0 0.0 0.0" rpy="0.0 0.0 0.0" />
-  </joint>
 </robot>
