Commit message: pix new

File: src/mapping/lio-sam/launch/include/config/pix_robot.urdf.xacro (robot description, xacro)
@@ -5,8 +5,15 @@
   <link name="ego_vehicle"></link>
   <!-- Sensor: lidar -->
-  <link name="hesai/pandar"></link>
+  <link name="lidar_top"></link>
   <joint name="lidar_joint" type="fixed">
     <parent link="ego_vehicle" />
     <child link="lidar_top" />
+    <origin xyz="0.0 0.0 0.0" rpy="0.0 0.0 0.0" />
+  </joint>
+  <!-- Sensor: gnss -->
+  <link name="gps_link"></link>
+  <joint name="gps_joint" type="fixed">
+    <parent link="ego_vehicle" />
+    <child link="gps_link" />
     <origin xyz="0.0 0.0 0.0" rpy="0.0 0.0 0.0" />
   </joint>
@@ -25,9 +32,9 @@
     <origin xyz="0.0 0.0 0.0" rpy="0.0 0.0 0.0" />
   </joint>
-  <!-- Sensor: odometry -->
-  <link name="ego_vehicle/odometry"></link>
-  <joint name="odometry_joint" type="fixed">
+  <!-- Sensor: imu -->
+  <link name="imu_link"></link>
+  <joint name="imu_pix_joint" type="fixed">
     <parent link="ego_vehicle" />
-    <child link="ego_vehicle/odometry" />
+    <child link="imu_link" />
     <origin xyz="0.0 0.0 0.0" rpy="0.0 0.0 0.0" />
   </joint>

File: src/mapping/liorf/launch/include/config/robot_pix.urdf.xacro (robot description, xacro)
@@ -7,5 +7,5 @@
     <parent link="base_link"/>
     <child link="chassis_link" />
-    <origin xyz="0 0 0" rpy="0 0 1.57079" />
+    <origin xyz="0 0 0" rpy="0 0 0" />
   </joint>
   <link name="ego_vehicle/imu"> </link>
@@ -13,4 +13,10 @@
     <parent link="chassis_link" />
     <child link="ego_vehicle/imu" />
+    <origin xyz="0 0 0" rpy="0 0 0" />
+  </joint>
+  <link name="imu_link"> </link>
+  <joint name="imu_pix_joint" type="fixed">
+    <parent link="chassis_link" />
+    <child link="imu_link" />
     <origin xyz="0 0 0" rpy="0 0 0" />
   </joint>
