Commit message: tracking error display

File: src/implementation/pix_model/urdf/pix_model.urdf (robot description, URDF)
Before this commit: robot Pix_molde, 3 links, 2 joints
Links:
- removed link base_link
- added link ego_vehicle, mass 36.9114288093113; collision mesh filename=package://pix_model/meshes/ego_vehicle.STL; visual mesh filename=package://pix_model/meshes/ego_vehicle.STL
- link imu_link: geometry collision mesh filename=package://pix_model/meshes/imu_link.STL; visual mesh filename=package://pix_model/meshes/imu_link.STL
- link laser: geometry collision mesh filename=package://pix_model/meshes/laser.STL; visual mesh filename=package://pix_model/meshes/laser.STL
Joints:
- joint imu_joint: parent base_link -> ego_vehicle
- joint laser_joint: parent base_link -> ego_vehicle

Commit message: anti-rollover

File: src/implementation/pix_model/urdf/pix_model.urdf (robot description, URDF)
Before this commit: robot pix_model, 3 links, 2 joints
Links:
- removed link base_link
- added link ego_vehicle, mass 36.9114288093113; collision mesh filename=package://pix_model/meshes/ego_vehicle.STL; visual mesh filename=package://pix_model/meshes/ego_vehicle.STL
Joints:
- joint imu_joint: parent base_link -> ego_vehicle
- joint laser_joint: parent base_link -> ego_vehicle
